File: Hyper7-Evo.kicad_sch (KiCad schematic)
At the start: 776 parts, among them J3 Conn_01x05, J4 Conn_01x03, J5 Conn_01x03, J6 Conn_01x05, J8 Conn_01x05

Commit message: dsfdsf
Parts:
- added J14, J15: Conn_01x04, Connector_PinHeader_2.54mm:PinHeader_1x04_P2.54mm_Vertical, symbol Connector_Generic:Conn_01x04
- added J16, J17: Conn_01x02, Connector_PinHeader_2.54mm:PinHeader_1x02_P2.54mm_Vertical, symbol Connector_Generic:Conn_01x02
Connections:
- net COL6: now also MX164.1
- net G_LED: now also J16.2 (Pin_2), J17.2 (Pin_2)
- net ROW0: now also J14.1 (Pin_1), J15.1 (Pin_1)
- net ROW1: now also J14.2 (Pin_2), J15.2 (Pin_2)
- net ROW2: now also J14.3 (Pin_3), J15.3 (Pin_3)
- net ROW3: now also J14.4 (Pin_4), J15.4 (Pin_4)
- net VDD: now also J16.1 (Pin_1), J17.1 (Pin_1)
