File: Hyper7-Evo.kicad_sch (KiCad schematic)
At the start: 780 parts, among them J14 Conn_01x04, J15 Conn_01x04, J16 Conn_01x02, J17 Conn_01x02, J3 Conn_01x05, J4 Conn_01x03, J5 Conn_01x03, J6 Conn_01x05, J8 Conn_01x05

Commit message: Completed board
Parts:
- added R10, R9: 5.1k, ergo-pw:R_0402_1005Metric, symbol ergo-pw:R-EU_R0603
- LED1, LED10, LED100, LED101, LED102, LED103, LED104, LED105, LED106, LED107, LED108, LED109, LED11, LED110, LED111, LED112, LED113, LED114, LED115, LED116, LED117, LED118, LED119, LED12, LED120, LED121, LED122, LED123, LED124, LED125, LED126, LED127, LED128, LED129, LED13, LED130, LED131, LED132, LED133, LED134, LED135, LED136, LED137, LED138, LED139, LED14, LED140, LED141, LED142, LED143, LED144, LED145, LED146, LED147, LED148, LED149, LED15, LED150, LED151, LED152, LED153, LED154, LED155, LED156, LED157, LED158, LED159, LED16, LED160, LED161, LED162, LED163, LED164, LED165, LED166, LED167, LED168, LED169, LED17, LED170, LED171, LED172, LED173, LED174, LED175, LED176, LED177, LED178, LED179, LED18, LED180, LED181, LED182, LED183, LED19, LED2, LED20, LED21, LED22, LED23, LED24, LED25, LED26, LED27, LED28, LED29, LED3, LED30, LED31, LED32, LED33, LED34, LED35, LED36, LED37, LED38, LED39, LED4, LED40, LED41, LED42, LED43, LED44, LED45, LED46, LED47, LED48, LED49, LED5, LED50, LED51, LED52, LED53, LED54, LED55, LED56, LED57, LED58, LED59, LED6, LED60, LED61, LED62, LED63, LED64, LED65, LED66, LED67, LED68, LED69, LED7, LED70, LED71, LED72, LED73, LED74, LED75, LED76, LED77, LED78, LED79, LED8, LED80, LED81, LED82, LED83, LED84, LED85, LED86, LED87, LED88, LED89, LED9, LED90, LED91, LED92, LED93, LED94, LED95, LED96, LED97, LED98, LED99: LCSC Part Not Available -> C3646935
Connections:
- net +3.3V: now also R10.2, R9.2
- net SCL: now also R10.1
- net SDA: now also R9.1
