File: nextgenplat.kicad_sch (KiCad schematic)
At the start: 35 parts, among them J1 XKB-USB-C16PIN, J2 BM02B-SRSS-TB, Q1 SI1308EDL-T1-GE3, Q2 SI1308EDL-T1-GE3, Q3 SI1308EDL-T1-GE3, U1 USBLC6-2P6, U10 74HC595, U2 XB3303ASOT23, U3 SiP32431DR3, U4 74HC595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

Commit message: dsfdsf
Parts:
- added J10, J11, J12, J13, J9: BM02B-SRSS-TB, ergo-pw:BM02B-SRSS-TB, symbol ergo-pw:BM02B-SRSS-TB
Connections:
- net +BATT: now also J10.2, J11.2, J12.2, J13.2, J9.2
- net -BATT: now also J10.1, J11.1, J12.1, J13.1, J9.1
Other:
- moved on the sheet: J2, R1
