File: ngpbase.kicad_sch (KiCad schematic)
At the start: 20 parts, among them J7 Conn_02x03_Odd_Even, U5 MDBT50Q-1MV2, U6 BQ24075RGT, Y1 Crystal

Commit message: Completed board
Parts:
- R14: value 1.8k -> 1.1k; LCSC Part C25871 -> C25860
- R15: value 1.8k -> 590; LCSC Part C25871 -> C2998181
Connections:
- net GND: now also U6.6 (EN1); no longer U6.5 (EN2)
- net VDD: now also U6.5 (EN2); no longer U6.6 (EN1)
Changed lines of the file:
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@@
 	(wire
 		(pts
+			(xy 179.07 101.6) (xy 179.07 100.965)
+		)
+		(stroke
+			(width 0)
+			(type default)
+		)
+	)
+	(wire
+		(pts
 			(xy 106.68 71.12) (xy 110.49 71.12)
 		)
@@
 	(wire
 		(pts
+			(xy 179.07 97.79) (xy 179.07 98.425)
+		)
+		(stroke
+			(width 0)
+			(type default)
+		)
+	)
+	(wire
+		(pts
 			(xy 106.68 35.56) (xy 118.11 35.56)
 		)
@@
 			)
 		)
-		(property "Value" "1.8k"
+		(property "Value" "590"
 			(at 182.372 117.475 0)
 			(effects
@@
 			)
 		)
-		(property "LCSC Part" "C25871"
+		(property "LCSC Part" "C2998181"
 			(at 179.07 113.665 0)
 			(effects
@@
 			)
 		)
-		(property "Value" "1.8k"
+		(property "Value" "1.1k"
 			(at 178.562 117.475 0)
 			(effects
@@
 			)
 		)
-		(property "LCSC Part" "C25871"
+		(property "LCSC Part" "C25860"
 			(at 175.26 113.665 0)
 			(effects
@@
 	(symbol
 		(lib_id "ergo-pw:VDD")
-		(at 179.07 98.425 90)
+		(at 179.07 101.6 90)
 		(unit 1)
 		(exclude_from_sim no)
@@
 		(fields_autoplaced yes)
 		(property "Reference" "#PWR055"
-			(at 182.88 98.425 0)
+			(at 182.88 101.6 0)
 			(effects
 				(font
@@
 		)
 		(property "Value" "VDD"
-			(at 175.26 98.425 90)
+			(at 175.26 101.6 90)
 			(effects
 				(font
@@
 		)
 		(property "Footprint" ""
-			(at 179.07 98.425 0)
+			(at 179.07 101.6 0)
 			(effects
 				(font
@@
 		)
 		(property "Datasheet" ""
-			(at 179.07 98.425 0)
+			(at 179.07 101.6 0)
 			(effects
 				(font
@@
 		)
 		(property "Description" ""
-			(at 179.07 98.425 0)
+			(at 179.07 101.6 0)
 			(effects
 				(font
@@
 	(symbol
 		(lib_id "ergo-pw:GND")
-		(at 179.07 100.965 270)
+		(at 179.07 97.79 270)
 		(unit 1)
 		(exclude_from_sim no)
@@
 		(dnp no)
 		(property "Reference" "#PWR056"
-			(at 172.72 100.965 0)
+			(at 172.72 97.79 0)
 			(effects
 				(font
@@
 		)
 		(property "Value" "GND"
-			(at 174.6758 101.092 0)
+			(at 174.6758 97.917 0)
 			(effects
 				(font
@@
 		)
 		(property "Footprint" ""
-			(at 179.07 100.965 0)
+			(at 179.07 97.79 0)
 			(effects
 				(font
@@
 		)
 		(property "Datasheet" ""
-			(at 179.07 100.965 0)
+			(at 179.07 97.79 0)
 			(effects
 				(font
@@
 		)
 		(property "Description" ""
-			(at 179.07 100.965 0)
+			(at 179.07 97.79 0)
 			(effects
 				(font
@@
 			)
 		)
-		(property "Description" "\n802.15.4, Bluetooth Bluetooth v5.2, Zigbee® Transceiver Module 2.36GHz ~ 2.5GHz Integrated, Chip Surface Mount\n"
+		(property "Description" "802.15.4, Bluetooth Bluetooth v5.2, Zigbee® Transceiver Module 2.36GHz ~ 2.5GHz Integrated, Chip Surface Mount"
 			(at 78.74 73.66 0)
 			(effects
